File: HW2/PCB_HW2/HW2.sch (EAGLE design)
At the start: 2 parts

Commit message: HW2_Sch_finished
Parts:
- removed PIC: (no value), HWlib:DIL28
- added C1, C2, C4, C5, C6: (no value), HWlib:C-US025-025X050
- added C3, C9: (no value), HWlib:CPOL-USE5-5
- added LED1, LED2: (no value), HWlib:LED3MM
- added PIC32: (no value), HWlib:DIL28-3
- added PICKIT3: (no value), HWlib:M05PTH
- added R1, R2, R3: (no value), HWlib:R-US_0207/10
- added RESONATOR: (no value), HWlib:M03PTH
- added U$2, U$4: PUSH_BUTTON, HWlib:PUSH_BUTTON
- added U$3: USB_MINI, HWlib:USB_MINI
Connections:
- new net +5V: C1.1, PIC32.15, U$1.2.VIN, U$3.5:VBUS
- new net N$1: PIC32.5, PICKIT3.5
- new net N$10: LED1.C, R2.1
- new net N$12: PIC32.10, RESONATOR.1
- new net N$13: LED2.A, PIC32.11
- new net N$14: LED2.C, R3.1
- new net N$16: PIC32.12, U$4.1
- new net N$2: PIC32.1, PICKIT3.1, R1.2, U$2.2
- new net N$20: C9.+, PIC32.20
- new net N$4: PIC32.14, U$3.2:ID
- new net N$5: PIC32.4, PICKIT3.4
- new net N$6: PIC32.21, U$3.3:D+
- new net N$7: PIC32.22, U$3.4:D-
- new net N$8: PIC32.9, RESONATOR.3
- net +3V3: now also C2.1, C3.+, C4.2, C5.1, C6.1, LED1.A, PIC32.13, PIC32.23, PIC32.28, PICKIT3.2, R1.1
- net GND: now also C1.2, C2.2, C3.-, C4.1, C5.2, C6.2, C9.-, PIC32.19, PIC32.27, PIC32.8, PICKIT3.3, R2.2, R3.2, RESONATOR.2, U$2.1, U$3.1:GND, U$4.2
Other:
- moved on the sheet: U$1

Commit message: PCB_Board
Parts:
- added M8_01, M8_02: (no value), HWlib:M08
- added U$5: SLIDE_SWITCH, HWlib:SLIDE_SWITCH
Connections:
- new net N$11: M8_01.2, PIC32.3
- new net N$15: M8_01.3, PIC32.6
- new net N$17: M8_01.4, PIC32.7
- new net N$18: M8_02.2, PIC32.25
- new net N$19: M8_02.1, PIC32.26
- new net N$21: M8_02.3, PIC32.24
- new net N$22: M8_02.4, PIC32.18
- new net N$23: M8_02.5, PIC32.17
- new net N$24: M8_02.6, PIC32.16
- new net N$3: U$3.5:VBUS, U$5.4
- new net N$9: M8_01.1, PIC32.2:A0
- net +3V3: now also M8_01.7
- net +5V: now also M8_02.7, U$5.3; no longer U$3.5:VBUS
- net GND: now also M8_01.8, M8_02.8
- net N$13: now also M8_01.5
- net N$16: now also M8_01.6
- net N$2: now also PIC32.1:!MCLR; no longer PIC32.1

Commit message: Ready to be checked before order
Parts:
- renumbered U$1 to 1
Changed lines of the file:
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@@
 </classes>
 <parts>
-<part name="U$1" library="HWlib" deviceset="MCP1702" device=""/>
+<part name="1" library="HWlib" deviceset="MCP1702" device=""/>
 <part name="GND1" library="HWlib" deviceset="GND" device=""/>
 <part name="+3V1" library="HWlib" deviceset="+3V3" device=""/>
@@
 <part name="M8_01" library="HWlib" deviceset="M08" device=""/>
 <part name="M8_02" library="HWlib" deviceset="M08" device=""/>
+<part name="GND12" library="HWlib" deviceset="GND" device=""/>
+<part name="+3V7" library="HWlib" deviceset="+3V3" device=""/>
+<part name="GND13" library="HWlib" deviceset="GND" device=""/>
+<part name="P+4" library="HWlib" deviceset="+5V" device=""/>
 </parts>
 <sheets>
@@
 </plain>
 <instances>
-<instance part="U$1" gate="G$1" x="-81.28" y="76.2"/>
+<instance part="1" gate="G$1" x="-81.28" y="76.2"/>
 <instance part="GND1" gate="1" x="-76.2" y="38.1" smashed="yes">
 <attribute name="VALUE" x="-78.74" y="35.56" size="1.778" layer="96"/>
@@
 <instance part="R3" gate="G$1" x="2.54" y="-45.72"/>
 <instance part="U$4" gate="G$1" x="25.4" y="-45.72"/>
-<instance part="GND3" gate="1" x="27.94" y="-55.88"/>
+<instance part="GND3" gate="1" x="27.94" y="-50.8"/>
 <instance part="P+3" gate="1" x="45.72" y="-12.7"/>
 <instance part="+3V5" gate="G$1" x="43.18" y="25.4"/>
-<instance part="GND10" gate="1" x="40.64" y="2.54"/>
+<instance part="GND10" gate="1" x="40.64" y="0"/>
 <instance part="C9" gate="G$1" x="55.88" y="-25.4"/>
 <instance part="GND11" gate="1" x="55.88" y="-38.1"/>
@@
 <instance part="M8_01" gate="G$1" x="-116.84" y="35.56"/>
 <instance part="M8_02" gate="G$1" x="-116.84" y="7.62"/>
+<instance part="GND12" gate="1" x="-101.6" y="50.8" smashed="yes">
+<attribute name="VALUE" x="-104.14" y="48.26" size="1.778" layer="96"/>
+</instance>
+<instance part="+3V7" gate="G$1" x="-91.44" y="53.34"/>
+<instance part="GND13" gate="1" x="-106.68" y="22.86" smashed="yes">
+<attribute name="VALUE" x="-109.22" y="20.32" size="1.778" layer="96"/>
+</instance>
+<instance part="P+4" gate="1" x="-99.06" y="22.86"/>
 </instances>
 <busses>
@@
 <net name="GND" class="0">
 <segment>
-<pinref part="U$1" gate="G$1" pin="1.GND"/>
+<pinref part="1" gate="G$1" pin="1.GND"/>
 <pinref part="GND1" gate="1" pin="GND"/>
 <wire x1="-76.2" y1="60.96" x2="-76.2" y2="58.42" width="0.1524" layer="91"/>
 <pinref part="C1" gate="G$1" pin="2"/>
-<wire x1="-76.2" y1="58.42" x2="-76.2" y2="50.8" width="0.1524" layer="91"/>
-<wire x1="-76.2" y1="50.8" x2="-76.2" y2="45.72" width="0.1524" layer="91"/>
-<wire x1="-76.2" y1="45.72" x2="-76.2" y2="40.64" width="0.1524" layer="91"/>
+<wire x1="-76.2" y1="58.42" x2="-76.2" y2="40.64" width="0.1524" layer="91"/>
 <wire x1="-101.6" y1="63.5" x2="-101.6" y2="58.42" width="0.1524" layer="91"/>
 <wire x1="-101.6" y1="58.42" x2="-76.2" y2="58.42" width="0.1524" layer="91"/>
@@
 <wire x1="-45.72" y1="40.64" x2="-76.2" y2="40.64" width="0.1524" layer="91"/>
 <junction x="-76.2" y="40.64"/>
-<pinref part="M8_01" gate="G$1" pin="8"/>
-<wire x1="-111.76" y1="45.72" x2="-76.2" y2="45.72" width="0.1524" layer="91"/>
-<junction x="-76.2" y="45.72"/>
-<pinref part="M8_02" gate="G$1" pin="8"/>
-<wire x1="-111.76" y1="17.78" x2="-86.36" y2="17.78" width="0.1524" layer="91"/>
-<wire x1="-86.36" y1="17.78" x2="-86.36" y2="50.8" width="0.1524" layer="91"/>
-<wire x1="-86.36" y1="50.8" x2="-76.2" y2="50.8" width="0.1524" layer="91"/>
-<junction x="-76.2" y="50.8"/>
 </segment>
 <segment>
@@
 <pinref part="U$4" gate="G$1" pin="2"/>
 <pinref part="GND3" gate="1" pin="GND"/>
-<wire x1="27.94" y1="-48.26" x2="27.94" y2="-53.34" width="0.1524" layer="91"/>
 </segment>
 <segment>
@@
 <wire x1="40.64" y1="12.7" x2="40.64" y2="7.62" width="0.1524" layer="91"/>
 <pinref part="C5" gate="G$1" pin="2"/>
-<wire x1="40.64" y1="7.62" x2="40.64" y2="5.08" width="0.1524" layer="91"/>
+<wire x1="40.64" y1="7.62" x2="40.64" y2="2.54" width="0.1524" layer="91"/>
 <wire x1="45.72" y1="7.62" x2="40.64" y2="7.62" width="0.1524" layer="91"/>
 <junction x="40.64" y="7.62"/>
@@
 <wire x1="55.88" y1="-30.48" x2="55.88" y2="-35.56" width="0.1524" layer="91"/>
 </segment>
+<segment>
+<pinref part="M8_01" gate="G$1" pin="8"/>
+<wire x1="-111.76" y1="45.72" x2="-106.68" y2="45.72" width="0.1524" layer="91"/>
+<wire x1="-106.68" y1="45.72" x2="-106.68" y2="55.88" width="0.1524" layer="91"/>
+<pinref part="GND12" gate="1" pin="GND"/>
+<wire x1="-106.68" y1="55.88" x2="-101.6" y2="55.88" width="0.1524" layer="91"/>
+<wire x1="-101.6" y1="55.88" x2="-101.6" y2="53.34" width="0.1524" layer="91"/>
+</segment>
+<segment>
+<pinref part="M8_02" gate="G$1" pin="8"/>
+<wire x1="-111.76" y1="17.78" x2="-109.22" y2="17.78" width="0.1524" layer="91"/>
+<wire x1="-109.22" y1="17.78" x2="-109.22" y2="25.4" width="0.1524" layer="91"/>
+<pinref part="GND13" gate="1" pin="GND"/>
+<wire x1="-109.22" y1="25.4" x2="-106.68" y2="25.4" width="0.1524" layer="91"/>
+</segment>
 </net>
 <net name="+3V3" class="0">
 <segment>
-<pinref part="U$1" gate="G$1" pin="3.VOUT"/>
+<pinref part="1" gate="G$1" pin="3.VOUT"/>
 <pinref part="+3V1" gate="G$1" pin="+3V3"/>
 <wire x1="-58.42" y1="76.2" x2="-50.8" y2="76.2" width="0.1524" layer="91"/>
@@
 <pinref part="C3" gate="G$1" pin="+"/>
 <wire x1="-45.72" y1="76.2" x2="-45.72" y2="50.8" width="0.1524" layer="91"/>
-<pinref part="M8_01" gate="G$1" pin="7"/>
-<wire x1="-111.76" y1="43.18" x2="-58.42" y2="43.18" width="0.1524" layer="91"/>
-<wire x1="-58.42" y1="43.18" x2="-58.42" y2="76.2" width="0.1524" layer="91"/>
-<junction x="-58.42" y="76.2"/>
 </segment>
 <segment>
@@
 <junction x="43.18" y="20.32"/>
 </segment>
+<segment>
+<pinref part="M8_01" gate="G$1" pin="7"/>
+<pinref part="+3V7" gate="G$1" pin="+3V3"/>
+<wire x1="-111.76" y1="43.18" x2="-91.44" y2="43.18" width="0.1524" layer="91"/>
+<wire x1="-91.44" y1="43.18" x2="-91.44" y2="50.8" width="0.1524" layer="91"/>
+</segment>
 </net>
 <net name="+5V" class="0">
 <segment>
+<pinref part="C1" gate="G$1" pin="1"/>
+<pinref part="1" gate="G$1" pin="2.VIN"/>
+<wire x1="-101.6" y1="76.2" x2="-93.98" y2="76.2" width="0.1524" layer="91"/>
+<wire x1="-101.6" y1="76.2" x2="-101.6" y2="71.12" width="0.1524" layer="91"/>
+<junction x="-101.6" y="76.2"/>
 <pinref part="P+1" gate="1" pin="+5V"/>
 <wire x1="-101.6" y1="91.44" x2="-101.6" y2="76.2" width="0.1524" layer="91"/>
-<pinref part="U$1" gate="G$1" pin="2.VIN"/>
-<wire x1="-101.6" y1="76.2" x2="-93.98" y2="76.2" width="0.1524" layer="91"/>
-<pinref part="C1" gate="G$1" pin="1"/>
-<wire x1="-101.6" y1="76.2" x2="-101.6" y2="71.12" width="0.1524" layer="91"/>
-<junction x="-101.6" y="76.2"/>
-<pinref part="M8_02" gate="G$1" pin="7"/>
-<wire x1="-111.76" y1="15.24" x2="-109.22" y2="15.24" width="0.1524" layer="91"/>
-<wire x1="-109.22" y1="15.24" x2="-109.22" y2="76.2" width="0.1524" layer="91"/>
-<wire x1="-109.22" y1="76.2" x2="-101.6" y2="76.2" width="0.1524" layer="91"/>
 </segment>
 <segment>
@@
 <pinref part="P+2" gate="1" pin="+5V"/>
 <wire x1="0" y1="48.26" x2="0" y2="58.42" width="0.1524" layer="91"/>
+</segment>
+<segment>
+<pinref part="M8_02" gate="G$1" pin="7"/>
+<pinref part="P+4" gate="1" pin="+5V"/>
+<wire x1="-111.76" y1="15.24" x2="-99.06" y2="15.24" width="0.1524" layer="91"/>
+<wire x1="-99.06" y1="15.24" x2="-99.06" y2="20.32" width="0.1524" layer="91"/>
 </segment>
 </net>
@@
 </segment>
 </net>
-<net name="N$24" class="0">
-<segment>
-<pinref part="PIC32" gate="G$1" pin="16"/>
-<wire x1="15.24" y1="-15.24" x2="17.78" y2="-15.24" width="0.1524" layer="91"/>
-<wire x1="17.78" y1="-15.24" x2="17.78" y2="-22.86" width="0.1524" layer="91"/>
-<wire x1="17.78" y1="-22.86" x2="-60.96" y2="-22.86" width="0.1524" layer="91"/>
-<wire x1="-60.96" y1="-22.86" x2="-60.96" y2="-27.94" width="0.1524" layer="91"/>
-<wire x1="-60.96" y1="-27.94" x2="-86.36" y2="-27.94" width="0.1524" layer="91"/>
-<wire x1="-86.36" y1="-27.94" x2="-86.36" y2="12.7" width="0.1524" layer="91"/>
-<pinref part="M8_02" gate="G$1" pin="6"/>
-<wire x1="-86.36" y1="12.7" x2="-111.76" y2="12.7" width="0.1524" layer="91"/>
-</segment>
-</net>
 <net name="N$3" class="0">
 <segment>
@@
 </segment>
 </net>
+<net name="N$26" class="0">
+<segment>
+<wire x1="17.78" y1="-15.24" x2="17.78" y2="-22.86" width="0.1524" layer="91"/>
+<pinref part="PIC32" gate="G$1" pin="16"/>
+<wire x1="15.24" y1="-15.24" x2="17.78" y2="-15.24" width="0.1524" layer="91"/>
+<wire x1="17.78" y1="-22.86" x2="-22.86" y2="-22.86" width="0.1524" layer="91"/>
+<wire x1="-22.86" y1="-22.86" x2="-22.86" y2="-33.02" width="0.1524" layer="91"/>
+<wire x1="-22.86" y1="-33.02" x2="-53.34" y2="-33.02" width="0.1524" layer="91"/>
+<wire x1="-53.34" y1="-33.02" x2="-53.34" y2="-27.94" width="0.1524" layer="91"/>
+<wire x1="-53.34" y1="-27.94" x2="-86.36" y2="-27.94" width="0.1524" layer="91"/>
+<wire x1="-86.36" y1="-27.94" x2="-86.36" y2="12.7" width="0.1524" layer="91"/>
+<pinref part="M8_02" gate="G$1" pin="6"/>
+<wire x1="-86.36" y1="12.7" x2="-111.76" y2="12.7" width="0.1524" layer="91"/>
+</segment>
+</net>
